File: circuito/poncho_nrf51822/poncho_nrf51822.kicad_pcb (KiCad board)
At the start: 2 copper layers, 86.4 x 61 mm, 7 parts, among them P1 CONN_5, P2 CONN_4

Commit message: placa
Parts:
- removed G***: Logo_EDU-CIAA, Poncho_Esqueleto:Logo_EDU-CIAA
- removed G***: LOGO, Poncho_Esqueleto:Logo_Poncho
- removed G101: Logo_OSHWA, Poncho_Esqueleto:Logo_OSHWA
- removed P1: CONN_5, Poncho_Modelos:bornier5
- removed P2: CONN_4, Poncho_Modelos:bornier4
- added C1: 100n, foot:C_0805_HandSoldering, B.Cu at (109.0, 111.0)
- added D1: LED, LEDs:LED_D5.0mm, F.Cu at (92.0, 118.0)
- added J1: CONN_01X18, Pin_Headers:Pin_Header_Straight_1x18_Pitch2.54mm, F.Cu at (84.0, 120.0)
- added J2: CONN_01X03, Pin_Headers:Pin_Header_Straight_1x03_Pitch2.54mm, F.Cu at (130.0, 99.0)
- added J3: CONN_02X05, Pin_Headers:Pin_Header_Straight_2x05_Pitch2.54mm, F.Cu at (131.0, 80.0)
- added J4: CONN_01X18, Pin_Headers:Pin_Header_Straight_1x18_Pitch2.54mm, F.Cu at (124.0, 77.0)
- added J5: CONN_01X02, Pin_Headers:Pin_Header_Straight_2x01_Pitch2.54mm, F.Cu at (128.0, 110.0)
- added J6: CONN_01X02, Pin_Headers:Pin_Header_Straight_2x01_Pitch2.54mm, F.Cu at (128.0, 105.0)
- added J7: CONN_01X02, Pin_Headers:Pin_Header_Straight_2x01_Pitch2.54mm, F.Cu at (128.0, 120.0)
- added J8: CONN_01X02, Pin_Headers:Pin_Header_Straight_2x01_Pitch2.54mm, F.Cu at (128.0, 115.0)
- added R1: 1k, foot:R_0805_HandSoldering, B.Cu at (103.0, 104.0)
- added R2: 10k, foot:R_0805_HandSoldering, B.Cu at (116.0, 119.0)
- added R3: 470R, foot:R_0805_HandSoldering, B.Cu at (100.0, 116.0)
- added SW1: SW_Push, Buttons_Switches_THT:SW_PUSH_6mm, F.Cu at (111.0, 115.0)
- added U1: yunjia_nrf51822, foot:yunjia_nrf51822, F.Cu at (93.0, 81.0)
Connections:
- XA1 pad 1: +3.3V -> /CiaaVcc
- XA1 pad 19: (no net) -> /CiaaSda
- XA1 pad 2: +5V -> (no net)
- XA1 pad 20: (no net) -> GND
- XA1 pad 21: (no net) -> /CiaaScl
- XA1 pad 22: (no net) -> GND
- XA1 pad 23: Net-(P1-Pad3) -> /CiaaRx
- XA1 pad 24: (no net) -> GND
- XA1 pad 25: Net-(P1-Pad4) -> /CiaaTx
- XA1 pad 26: (no net) -> GND
- XA1 pad 28: (no net) -> GND
- XA1 pad 30: (no net) -> GND
- XA1 pad 32: (no net) -> GND
- XA1 pad 38: (no net) -> GND
- XA1 pad 4: (no net) -> GND
- XA1 pad 40: (no net) -> GND
- XA1 pad 42: +5VP -> (no net)
- XA1 pad 51: (no net) -> GND
- XA1 pad 53: (no net) -> GND
- XA1 pad 57: (no net) -> GND
- XA1 pad 59: (no net) -> GND
- XA1 pad 65: (no net) -> GND
- XA1 pad 67: (no net) -> GND
- XA1 pad 72: Net-(P2-Pad3) -> /GPIO1
- XA1 pad 74: Net-(P2-Pad2) -> /GPIO2
- XA1 pad 76: (no net) -> /GPIO3
- XA1 pad 78: (no net) -> /GPIO4
- XA1 pad 80: (no net) -> /GPIO5
Routing:
- net GND: track 130.8 -> 388.3 mm, vias 0 -> 2
- net +3.3V: track 34.8 -> 139.6 mm
- net +5VP: track 73.3 -> 0.00 mm
- net Net-(P1-Pad4): track 60.1 -> 0.00 mm
- net Net-(P1-Pad3): track 54.7 -> 0.00 mm
- net /BtnCont: track 0.00 -> 52.8 mm
- net /LedCont: track 0.00 -> 51.8 mm
- net /GPIO5: track 0.00 -> 51.3 mm, vias 0 -> 1
- net /GPIO4: track 0.00 -> 46.0 mm, vias 0 -> 1
- net /P13: track 0.00 -> 43.5 mm
- net Net-(P2-Pad3): track 43.4 -> 0.00 mm
- net /n51Rx: track 0.00 -> 43.4 mm
- net /GPIO2: track 0.00 -> 41.8 mm, vias 0 -> 1
- net /GPIO3: track 0.00 -> 41.6 mm, vias 0 -> 1
- net /GPIO1: track 0.00 -> 40.7 mm, vias 0 -> 1
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- added copper zone on B.Cu, net GND
- added copper zone on F.Cu, net GND
Other:
- net class Default: via_dia 0.6 -> 2.5; via_drill 0.4 -> 0.8
- board text removed: "Borrar (Footprint MP1) la Plantilla-EDU-CIAA al finalizar el posicionamiento y definido el borde de PCB."
- board text removed: "Diseño simple faz. Sin requerimientos especiales."
- board text removed: "Editar el rótulo"
- board text removed: "Editar el stackup para reflejar cantidad de capas, si se han realizado cálculos de impedancia o si es relevante para el funcionamiento."
- board text removed: "PONCHO CHICO"
- board text removed: "PONCHO CHICO http://www.proyecto-ciaa.com.ar/"
- board text removed: "Para un diseño nuevo luego de modificar el esquemático: 1)Seleccionar el bloque del PCB y cotas. (click-drag-release). 2)Opción de borrar bloque (Botón derecho). 3)Marcar todo menos locked footprints (MP1 y XA1) 4) Aceptar. 5) Volver a cargar el netlist."
- board text removed: "STACK-UP"
- board text removed: "Se sugiere colocar código de Poncho en cobre, serigrafía y rótulo."
- board text removed: "www.proyecto-ciaa.com.ar"
