File: circuito/poncho_nrf51822/poncho_nrf51822.kicad_pcb (KiCad board)
At the start: 2 copper layers, 86.4 x 61 mm, 17 parts, among them J1 CONN_01X18, J2 CONN_01X03, J3 CONN_02X05, J4 CONN_01X18, J5 CONN_01X02, J6 CONN_01X02, J7 CONN_01X02, J8 CONN_01X02, SW1 SW_Push, U1 yunjia_nrf51822

Commit message: poncho echo
Parts:
- C1: footprint foot:C_0805_HandSoldering -> footprints:C_0805_HandSoldering
- D1: footprint LEDs:LED_D5.0mm -> footprints:LED_D5.0mm
- J1, J4: footprint Pin_Headers:Pin_Header_Straight_1x18_Pitch2.54mm -> footprints:Pin_Header_Straight_1x18_Pitch2.54mm
- J2: footprint Pin_Headers:Pin_Header_Straight_1x03_Pitch2.54mm -> footprints:Pin_Header_Straight_1x03_Pitch2.54mm
- J3: footprint Pin_Headers:Pin_Header_Straight_2x05_Pitch2.54mm -> footprints:Pin_Header_Straight_2x05_Pitch2.54mm
- J5, J6, J7, J8: footprint Pin_Headers:Pin_Header_Straight_2x01_Pitch2.54mm -> footprints:Pin_Header_Straight_2x01_Pitch2.54mm
- R1, R2, R3: footprint foot:R_0805_HandSoldering -> footprints:R_0805_HandSoldering
- SW1: footprint Buttons_Switches_THT:SW_PUSH_6mm -> footprints:SW_PUSH_6mm
- U1: footprint foot:yunjia_nrf51822 -> footprints:yunjia_nrf51822
- XA1: footprint Poncho_Esqueleto:Conn_Poncho_Chico -> footprints:Conn_Poncho_Chico
- moved J7 1.16 mm to (129.2, 119.9)
- moved J6 1.16 mm to (129.2, 104.9)
- moved J8 1.16 mm to (129.2, 115.1)
- moved J5 1.16 mm to (129.2, 110.0)
Connections:
- J3 pad 1: (no net) -> Net-(J3-Pad1)
- J3 pad 10: (no net) -> Net-(J3-Pad10)
- J3 pad 5: (no net) -> Net-(J3-Pad5)
- J3 pad 9: (no net) -> Net-(J3-Pad9)
- XA1 pad 2: (no net) -> Net-(XA1-Pad2)
- XA1 pad 41: (no net) -> Net-(XA1-Pad41)
- XA1 pad 42: (no net) -> Net-(XA1-Pad42)
- XA1 pad 69: (no net) -> Net-(XA1-Pad69)
- XA1 pad 71: (no net) -> Net-(XA1-Pad71)
- XA1 pad 73: (no net) -> Net-(XA1-Pad73)
- XA1 pad 75: (no net) -> Net-(XA1-Pad75)
Routing:
- net /n51Sda: track 25.5 -> 29.9 mm
- net +3.3V: track 139.6 -> 143.6 mm
- net /P10: track 14.1 -> 17.1 mm
- net /P12: track 12.7 -> 15.0 mm
- net /P14: track 12.4 -> 14.6 mm
- net /n51Tx: track 35.0 -> 36.9 mm
- net GND: track 388.3 -> 390.0 mm
- net /n51Scl: track 31.6 -> 33.2 mm
- net /GPIO5: track 51.3 -> 53.0 mm
- net /CiaaSda: track 12.4 -> 10.9 mm
- net /LedCont: track 51.8 -> 53.4 mm
- net /CiaaScl: track 13.1 -> 11.9 mm
- net /SWCLK: track 35.0 -> 36.2 mm
- net /P06: track 15.7 -> 16.7 mm
- net /P08: track 15.3 -> 16.2 mm
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Other:
- net class Default: clearance 0.508 -> 0.3
- rule trace_clearance: 0.508 -> 0.3

Commit message: poncho echo
Routing:
- net GND: track 390.0 -> 394.9 mm, vias 2 -> 3
