File: circuito/poncho_nrf51822/_autosave-poncho_nrf51822.kicad_pcb (KiCad board)
At the start: 2 copper layers, 86.4 x 61 mm, 17 parts, among them J1 CONN_01X18, J2 CONN_01X03, J3 CONN_02X05, J4 CONN_01X18, J5 CONN_01X02, J6 CONN_01X02, J7 CONN_01X02, J8 CONN_01X02, SW1 SW_Push, U1 yunjia_nrf51822

Commit message: WIP
Connections:
- net /BtnCont renamed /BtnCont(P15)
- net /GPIO1 renamed /GPIO1(P01)
- net /GPIO2 renamed /GPIO2(P03)
- net /GPIO3 renamed /GPIO3(P04)
- net /GPIO4 renamed /GPIO4(P02)
- net /GPIO5 renamed /GPIO5(P00)
- net /LedCont renamed /LedCont(P29)
- net /n51Rx renamed /n51Rx(P11)
- net /n51Scl renamed /n51Scl(P07)
- net /n51Sda renamed /n51Sda(P05)
- net /n51Tx renamed /n51Tx(P09)
