File: circuito/poncho_nrf51822/poncho_nrf51822.sch (KiCad schematic (older format))
At the start: 5 parts

Commit message: placa
Parts:
- added C1: 100n, footprints:C_0805_HandSoldering, symbol C
- added D1: LED, footprints:LED_D5.0mm, symbol LED
- added J2: CONN_01X03, footprints:Pin_Header_Straight_1x03_Pitch2.54mm, symbol CONN_01X03
- added J3: CONN_02X05, footprints:Pin_Header_Straight_2x05_Pitch2.54mm, symbol CONN_02X05
- added J5, J6, J7, J8: CONN_01X02, footprints:Pin_Header_Straight_2x01_Pitch2.54mm, symbol CONN_01X02
- added R1: 1k, footprints:R_0805_HandSoldering, symbol R
- added R2: 10k, footprints:R_0805_HandSoldering, symbol R
- added R3: 470R, footprints:R_0805_HandSoldering, symbol R
- added SW1: SW_Push, footprints:SW_PUSH_6mm, symbol SW_Push
- J1, J4: renamed from J?; footprint (none) -> footprints:Pin_Header_Straight_1x18_Pitch2.54mm
- U1: renamed from U?; footprint (none) -> footprints:yunjia_nrf51822
- XA1: footprint Poncho_Esqueleto:Conn_Poncho_Chico -> footprints:Conn_Poncho_Chico
- XA1: footprint (none) -> footprints:Conn_Poncho_Chico
- XA1: renamed from XA?; footprint (none) -> footprints:Conn_Poncho_Chico
Connections:
- net +3.3V: now also J1.9 (P9), U1.11 (VDD), J2.2 (P2), R2.1; no longer XA1.1 (+3.3V)
- net +5V: no longer XA1.2 (+5V)
- net GND: now also J1.14 (P14), J1.2 (P2), U1.1 (GND), U1.12 (GND), XA1.20 (GND), XA1.22 (GND), XA1.24 (GND), XA1.26 (GND), XA1.28 (GND), XA1.30 (GND), XA1.32 (GND), XA1.38 (GND), XA1.4 (GND), XA1.40 (GND), XA1.51 (GND), XA1.53 (GND), XA1.57 (GND), XA1.59 (GND), XA1.65 (GND), XA1.67 (GND), C1.2, D1.1 (K), J3.3 (P3), J3.4 (P4), SW1.2
- net CiaaRx: now reaches XA1.23 (RXD)
- net CiaaRx: now also J8.2 (P2)
- net CiaaTx: now reaches XA1.25 (TXD)
- net CiaaTx: now also J7.2 (P2)
- net GPIO1: now reaches XA1.72 (GPIO1)
- net GPIO1: now also J1.7 (P7), U1.15 (P0.01)
- net GPIO2: now reaches XA1.74 (GPIO3)
- net GPIO2: now also J1.6 (P6), U1.17 (P0.03)
- net GPIO3: now reaches XA1.76 (GPIO5)
- net GPIO3: now also J1.5 (P5), U1.18 (P0.04)
- net GPIO4: now reaches XA1.78 (GPIO7)
- net GPIO4: now also J1.4 (P4), U1.16 (P0.02)
- net GPIO5: now reaches XA1.80 (GPIO8)
- net GPIO5: now also J1.3 (P3), U1.14 (P0.00)
- net LedCont: now reaches U1.10 (P0.29)
- net LedCont: now also J1.1 (P1), R3.2
- net P30: now reaches U1.13 (P0.30)
- net P30: now also J1.8 (P8)
- net P18: now reaches U1.19 (P0.18)
- net P18: now also J4.4 (P4)
- net P21: now reaches U1.2 (P0.21)
- net P21: now also J1.15 (P15)
- net P20: now reaches U1.20 (P0.20)
- net P20: now also J4.5 (P5)
- net P17: now reaches U1.21 (P0.17)
- net P17: now also J4.3 (P3)
- net P19: now reaches U1.22 (P0.19)
- net P19: now also J4.6 (P6)
- net SWDIO: now reaches U1.23 (SWDIO)
- net SWDIO: now also J4.2 (P2), J3.2 (P2)
- net SWCLK: now reaches U1.24 (SWCLK)
- net SWCLK: now also J4.7 (P7), J3.6 (P6)
- net BtnCont: now reaches U1.25 (P0.15)
- net BtnCont: now also J4.1 (P1), R1.1
- net P16: now reaches U1.26 (P0.16)
- net P16: now also J4.8 (P8)
- net P13: now reaches U1.27 (P0.13)
- net P13: now also J4.18 (P18)
- net P14: now reaches U1.28 (P0.14)
- net P14: now also J4.9 (P9)
- net n51Rx: now reaches U1.29 (P0.11)
- net n51Rx: now also J4.17 (P17), J7.1 (P1)
- net P22: now reaches U1.3 (P0.22)
- net P22: now also J1.13 (P13)
- net P12: now reaches U1.30 (P0.12)
- net P12: now also J4.10 (P10)
- net n51Tx: now reaches U1.31 (P0.09)
- net n51Tx: now also J4.16 (P16), J8.1 (P1)
- net P10: now reaches U1.32 (P0.10)
- net P10: now also J4.11 (P11)
- net n51Scl: now reaches U1.33 (P0.07)
- net n51Scl: now also J4.15 (P15), J5.1 (P1)
- net P08: now reaches U1.34 (P0.08)
- net P08: now also J4.12 (P12)
- net n51Sda: now reaches U1.35 (P0.05)
- net n51Sda: now also J4.14 (P14), J6.1 (P1)
- net P06: now reaches U1.36 (P0.06)
- net P06: now also J4.13 (P13)
- net P23: now reaches U1.4 (P0.23)
- net P23: now also J1.16 (P16)
- net P24: now reaches U1.5 (P0.24)
- net P24: now also J1.12 (P12)
- net P25: now reaches U1.6 (P0.25)
- net P25: now also J1.17 (P17)
- net P26: now reaches U1.7 (P0.26)
- net P26: now also J1.11 (P11)
- net P27: now reaches U1.8 (P0.27)
- net P27: now also J1.18 (P18)
- net P28: now reaches U1.9 (P0.28)
- net P28: now also J1.10 (P10)
- net CiaaSda: now reaches XA1.19 (SDA)
- net CiaaSda: now also J6.2 (P2)
- net CiaaScl: now reaches XA1.21 (SCL)
- net CiaaScl: now also J5.2 (P2)
- net +5VP: no longer names the net of XA1.42 (+5V)
- new net: D1.2 (A), R3.1
- new net: C1.1, R1.2, R2.2, SW1.1
- new net CiaaVcc: J2.3 (P3), XA1.1 (+3.3V)
- new net ProgVcc: J2.1 (P1), J3.7 (P7), J3.8 (P8)
- no-connect marks 17 -> 11
Other:
- moved on the sheet: J1, J4, XA1A, XA1E, XA1F, XA1K

Commit message: WIP
Connections:
- net BtnCont renamed BtnCont(P15)
- net GPIO1 renamed GPIO1(P01)
- net GPIO2 renamed GPIO2(P03)
- net GPIO3 renamed GPIO3(P04)
- net GPIO4 renamed GPIO4(P02)
- net GPIO5 renamed GPIO5(P00)
- net LedCont renamed LedCont(P29)
- net n51Rx renamed n51Rx(P11)
- net n51Scl renamed n51Scl(P07)
- net n51Sda renamed n51Sda(P05)
- net n51Tx renamed n51Tx(P09)
Other:
- moved on the sheet: J1, J4, XA1K
